Commit message: urdf made with wheels

File: trunk/ROS/catkin_ws/src/oculus2wd/oculus2wd.urdf (robot description, URDF)
Before this commit: robot multipleshapes, 2 links, 1 joints
Links:
- removed link right_leg
- added link left_motor; visual cylinder length=0.008 radius=0.066
- added link right_motor; visual cylinder length=0.008 radius=0.066
- added link stand_link; visual box size=0.045 .095 .23
- link base_link: geometry visual box size=.26 .28 .06
Joints:
- removed joint base_to_right_leg
- added joint base_to_left_motor: type fixed, parent base_link, child left_motor
- added joint base_to_right_motor: type fixed, parent base_link, child right_motor
- added joint base_to_stand: type fixed, parent base_link, child stand_link
