Commit message: orange_on_wheels.urdf sizes updated

File: nodes/hubee/catkin_ws/orange_on_wheels.urdf (robot description, URDF)
Before this commit: robot orange_on_wheels, 6 links, 5 joints
Links:
- link base_link: geometry visual box size=0.21 0.17 0.29
- link fwheel: geometry visual cylinder length=0.014 radius=0.033
- link lwheel: geometry visual cylinder length=0.025 radius=0.0325
- link rwheel: geometry visual cylinder length=0.025 radius=0.0325
Joints:
- joint base_to_fwheel: origin xyz=0.13 0 0.02 rpy=0 0 0 -> xyz=0.9 0 0.02 rpy=0 0 0
