Commit message: urdf edited

File: ROS/custom_src/orange_on_wheels/orange_on_wheels.urdf (robot description, URDF)
Before this commit: robot orange_on_wheels, 6 links, 5 joints
Links:
- removed link fwheel
- removed link fwheel_attach
- removed link scanner
- added link back_wheel; visual cylinder length=0.014 radius=0.0165
- added link back_wheel_attach; visual box size=0.02 0.025 0.02
- added link imu; visual box size=0.01 0.01 0.01
- added link imu_frame; visual box size=0.01 0.12 0.255
- added link ultrasound; visual box size=0.015 0.045 0.015
- link base_link: geometry visual box size=0.21 0.17 0.003
Joints:
- removed joint base_to_fattach
- removed joint base_to_fwheel
- added joint back_wheel_attach_to_back_wheel: type fixed, parent back_wheel_attach, child back_wheel, origin xyz=0 0 -0.02 rpy=0 0 0
- added joint base_to_back_attach: type fixed, parent base_link, child back_wheel_attach, origin xyz=-0.08 0 0 rpy=0 0 0
- added joint base_to_imu_frame: type fixed, parent base_link, child imu_frame, origin xyz=0.04 0 0.135 rpy=0 0 0
- added joint imu_frame_to_imu: type fixed, parent imu_frame, child imu, origin xyz=0 0 0.1 rpy=0 0 0
- joint base_to_lwheel: origin xyz=0 0.115 0.046 rpy=1.5708 0 0 -> xyz=0 0.115 -0.01 rpy=1.5708 0 0
- joint base_to_rwheel: origin xyz=0 -0.115 0.046 rpy=-1.5708 0 0 -> xyz=0 -0.115 -0.01 rpy=-1.5708 0 0
- joint base_to_scanner: child scanner -> ultrasound; origin xyz=0.105 0 0.22 rpy=0 0 0 -> xyz=0.095 0 0.007 rpy=0 0 0

Commit message: third party frames added

File: ROS/custom_src/orange_on_wheels/orange_on_wheels.urdf (robot description, URDF)
Before this commit: robot orange_on_wheels, 8 links, 7 joints
Links:
- removed link imu_frame
- added link base_footprint; visual box size=0.01 0.12 0.255
- added link odom
Joints:
- removed joint base_to_imu_frame
- removed joint imu_frame_to_imu
- added joint base_footprint_to_imu: type fixed, parent base_footprint, child imu, origin xyz=0 0 0.1 rpy=0 0 0
- added joint base_to_base_footprint: type fixed, parent base_link, child base_footprint, origin xyz=0.04 0 0.135 rpy=0 0 0
- added joint base_to_odom: type fixed, parent base_link, child odom, origin xyz=0 0 0 rpy=0 0 0

Commit message: odom -> parent

File: ROS/custom_src/orange_on_wheels/orange_on_wheels.urdf (robot description, URDF)
Before this commit: robot orange_on_wheels, 9 links, 8 joints
Joints:
- joint base_to_odom: child odom -> base_link; parent base_link -> odom

Commit message: back_ultrasound added to urdf

File: ROS/custom_src/orange_on_wheels/orange_on_wheels.urdf (robot description, URDF)
Before this commit: robot orange_on_wheels, 9 links, 8 joints
Links:
- added link back_ultrasound; visual box size=0.015 0.045 0.015
Joints:
- added joint base_to_back_scanner: type fixed, parent base_link, child back_ultrasound, origin xyz=-0.095 0 0.007 rpy=0 0 0

Commit message: adjustments in urdf

File: ROS/custom_src/orange_on_wheels/orange_on_wheels.urdf (robot description, URDF)
Before this commit: robot orange_on_wheels, 10 links, 9 joints
Joints:
- joint base_to_back_scanner: origin xyz=-0.095 0 0.007 rpy=0 0 0 -> xyz=-0.095 0 0.007 rpy=0 0 3.14

Commit message: distance between wheels is 14 cm, not 23

File: ROS/custom_src/orange_on_wheels/orange_on_wheels.urdf (robot description, URDF)
Before this commit: robot orange_on_wheels, 10 links, 9 joints
Joints:
- joint base_to_lwheel: origin xyz=0 0.115 -0.01 rpy=1.5708 0 0 -> xyz=0 0.07 -0.01 rpy=1.5708 0 0
- joint base_to_rwheel: origin xyz=0 -0.115 -0.01 rpy=-1.5708 0 0 -> xyz=0 -0.07 -0.01 rpy=-1.5708 0 0
