Commit message: robot model in xacro

File: ROS/custom_src/orange_on_track/orange_on_track.xacro (robot description, xacro)
@@ -20,6 +20,10 @@
 	<xacro:property name="wheel_width" value="0.021" />
 	<xacro:property name="wheel_x_offset" value="${green_plate_length / 2 - wheel_radius}" />
-	<xacro:property name="wheel_y_offset" value="${green_plate_widths / 2 + wheel_width / 2}" />
+	<xacro:property name="wheel_y_offset" value="${green_plate_width / 2 + wheel_width / 2}" />
 	<xacro:property name="wheel_color" value="0 0 0 1" />
+	<xacro:property name="header_width" value="0.08" />
+	<xacro:property name="header_length" value="0.04" />
+	<xacro:property name="header_height" value="0.006" />
+	<xacro:property name="header_x_offset" value="0.10" />
 	<link name="base_link">
 		<visual>
@@ -97,4 +101,20 @@
 		<origin xyz="0 ${-white_plate_width / 2} ${-stand_length / 2}" rpy="0 0 0"/>
 	</joint>
+	<link name="header">
+		<visual>
+			<geometry>
+				<box size="${header_length} ${header_width} ${header_height}"/>
+			</geometry>
+			<origin xyz="0 0 0" rpy="0 0 0"/>
+			<material name="white">
+				<color rgba="0 0 0.5 0.1"/>
+			</material>
+		</visual>
+	</link>
+	<joint name="white_plate_to_header" type="fixed">
+		<parent link="white_plate"/>
+		<child link="header"/>
+		<origin xyz="${header_x_offset} 0 ${white_plate_height}" rpy="0 0 0"/>
+	</joint>
 	<link name="left_rear_wheel">
 		<visual>

Commit message: macro track added to xacro

File: ROS/custom_src/orange_on_track/orange_on_track.xacro (robot description, xacro)
@@ -117,67 +117,39 @@
 		<origin xyz="${header_x_offset} 0 ${white_plate_height}" rpy="0 0 0"/>
 	</joint>
-	<link name="left_rear_wheel">
-		<visual>
-			<geometry>
-				<cylinder length="${wheel_width}" radius="${wheel_radius}"/>
-			</geometry>
-			<origin rpy="0 0 0" xyz="0 0 0"/>
-			<material name="black">
-				<color rgba="${wheel_color}"/>
-			</material>
-		</visual>
-	</link>
-	<link name="right_rear_wheel">
-		<visual>
-			<geometry>
-				<cylinder length="${wheel_width}" radius="${wheel_radius}"/>
-			</geometry>
-			<origin rpy="0 0 0" xyz="0 0 0"/>
-			<material name="black">
-				<color rgba="${wheel_color}"/>
-			</material>
-		</visual>
-	</link>
-	<link name="left_fwd_wheel">
-		<visual>
-			<geometry>
-				<cylinder length="${wheel_width}" radius="${wheel_radius}"/>
-			</geometry>
-			<origin rpy="0 0 0" xyz="0 0 0"/>
-			<material name="black">
-				<color rgba="${wheel_color}"/>
-			</material>
-		</visual>
-	</link>
-	<link name="right_fwd_wheel">
-		<visual>
-			<geometry>
-				<cylinder length="${wheel_width}" radius="${wheel_radius}"/>
-			</geometry>
-			<origin rpy="0 0 0" xyz="0 0 0"/>
-			<material name="black">
-				<color rgba="${wheel_color}"/>
-			</material>
-		</visual>
-	</link>
-	<joint name="base_to_left_rear_wheel" type="fixed">
-		<parent link="base_link"/>
-		<child link="left_rear_wheel"/>
-		<origin xyz="${-wheel_x_offset} ${-wheel_y_offset} 0" rpy="${pi / 2} 0 0"/>
-	</joint>
-	<joint name="base_to_right_rear_wheel" type="fixed">
-		<parent link="base_link"/>
-		<child link="right_rear_wheel"/>
-		<origin xyz="{-wheel_x_offset} ${wheel_y_offset} 0" rpy="${pi / 2} 0 0"/>
-	</joint>
-	<joint name="base_to_left_fwd_wheel" type="fixed">
-		<parent link="base_link"/>
-		<child link="left_fwd_wheel"/>
-		<origin xyz="${wheel_x_offset} ${-wheel_y_offset} 0" rpy="${pi / 2} 0 0"/>
-	</joint>
-	<joint name="base_to_right_fwd_wheel" type="fixed">
-		<parent link="base_link"/>
-		<child link="right_fwd_wheel"/>
-		<origin xyz="{wheel_x_offset} ${wheel_y_offset} 0" rpy="${pi / 2} 0 0"/>
-	</joint>
+	<xacro:macro name="track" params="prefix reflect">
+		<link name="${prefix}_rear_wheel">
+			<visual>
+				<geometry>
+					<cylinder length="${wheel_width}" radius="${wheel_radius}"/>
+				</geometry>
+				<origin rpy="0 0 0" xyz="0 0 0"/>
+				<material name="black">
+					<color rgba="${wheel_color}"/>
+				</material>
+			</visual>
+		</link>
+		<link name="${prefix}_fwd_wheel">
+			<visual>
+				<geometry>
+					<cylinder length="${wheel_width}" radius="${wheel_radius}"/>
+				</geometry>
+				<origin rpy="0 0 0" xyz="0 0 0"/>
+				<material name="black">
+					<color rgba="${wheel_color}"/>
+				</material>
+			</visual>
+		</link>
+		<joint name="base_to_${prefix}_rear_wheel" type="fixed">
+			<parent link="base_link"/>
+			<child link="${prefix}_rear_wheel"/>
+			<origin xyz="${-wheel_x_offset} ${reflect*wheel_y_offset} 0" rpy="${pi / 2} 0 0"/>
+		</joint>
+		<joint name="base_to_${prefix}_fwd_wheel" type="fixed">
+			<parent link="base_link"/>
+			<child link="${prefix}_fwd_wheel"/>
+			<origin xyz="${wheel_x_offset} ${reflect*wheel_y_offset} 0" rpy="${pi / 2} 0 0"/>
+		</joint>
+	</xacro:macro>
+	<xacro:track prefix="right" reflect="1" />
+	<xacro:track prefix="left" reflect="-1" />
 </robot>

Commit message: more gazebo stuff added

File: ROS/custom_src/orange_on_track/orange_on_track.xacro (robot description, xacro)
@@ -140,14 +140,23 @@
 			</visual>
 		</link>
-		<joint name="base_to_${prefix}_rear_wheel" type="fixed">
+		<joint name="base_to_${prefix}_rear_wheel" type="continuous">
 			<parent link="base_link"/>
 			<child link="${prefix}_rear_wheel"/>
 			<origin xyz="${-wheel_x_offset} ${reflect*wheel_y_offset} 0" rpy="${pi / 2} 0 0"/>
 		</joint>
-		<joint name="base_to_${prefix}_fwd_wheel" type="fixed">
+		<joint name="base_to_${prefix}_fwd_wheel" type="continuous">
 			<parent link="base_link"/>
 			<child link="${prefix}_fwd_wheel"/>
 			<origin xyz="${wheel_x_offset} ${reflect*wheel_y_offset} 0" rpy="${pi / 2} 0 0"/>
 		</joint>
+		<transmission name="base_to_${prefix}_rear_trans">
+			<type>transmission_interface/SimpleTransmission</type>
+			<actuator name="base_to_${prefix}_rear_motor">
+				<mechanicalReduction>1</mechanicalReduction>
+			</actuator>
+			<joint name="base_to_${prefix}_rear_wheel">
+				<hardwareInterface>PositionJointInterface</hardwareInterface>
+			</joint>
+		</transmission>
 	</xacro:macro>
 	<xacro:track prefix="right" reflect="1" />

Commit message: visual fixing

File: ROS/custom_src/orange_on_track/orange_on_track.xacro (robot description, xacro)
@@ -1,8 +1,7 @@
 <?xml version="1.0"?>
 <robot xmlns:xacro="http://www.ros.org/wiki/xacro" name="orange_on_track">
-	<xacro:property name="pi" value="3.1416" />
 	<xacro:property name="base_width" value="0.105" />
 	<xacro:property name="base_length" value="0.17" />
-	<xacro:property name="base_height" value="0.046" />
+	<xacro:property name="base_height" value="0.043" />
 	<xacro:property name="green_plate_width" value="0.105" />
 	<xacro:property name="green_plate_length" value="0.17" />
@@ -11,10 +10,10 @@
 	<xacro:property name="white_plate_width" value="0.20" />
 	<xacro:property name="white_plate_length" value="0.245" />
-	<xacro:property name="white_plate_height" value="0.019" />
-	<xacro:property name="white_plate_x_offset" value="-0.025" />
+	<xacro:property name="white_plate_height" value="0.009" />
+	<xacro:property name="white_plate_x_offset" value="-0.015" />
 	<xacro:property name="white_plate_z_offset" value="0.029" />
-	<xacro:property name="stand_width" value="0.05" />
-	<xacro:property name="stand_length" value="0.195" />
-	<xacro:property name="stand_height" value="0.002" />
+	<xacro:property name="stand_width" value="0.002" />
+	<xacro:property name="stand_length" value="0.05" />
+	<xacro:property name="stand_height" value="0.195" />
 	<xacro:property name="wheel_radius" value="0.0235" />
 	<xacro:property name="wheel_width" value="0.021" />
@@ -24,14 +23,15 @@
 	<xacro:property name="header_width" value="0.08" />
 	<xacro:property name="header_length" value="0.04" />
-	<xacro:property name="header_height" value="0.006" />
+	<xacro:property name="header_height" value="0.06" />
 	<xacro:property name="header_x_offset" value="0.10" />
+	<xacro:property name="header_z_offset" value="0.06" />
 	<link name="base_link">
 		<visual>
 			<geometry>
-				<box size="${white_plate_width} ${white_plate_length} 0.009"/>
+				<box size="${base_length} ${base_width} ${base_height}"/>
 			</geometry>
 			<origin xyz="0 0 0" rpy="0 0 0"/>
-			<material name="white">
-				<color rgba="1 1 1 0.5"/>
+			<material name="gray">
+				<color rgba="0.5 0.5 0.5 0"/>
 			</material>
 		</visual>
@@ -45,8 +45,8 @@
 		<visual>
 			<geometry>
-				<box size="${green_plate_width} ${green_plate_length} ${green_plate_height}"/>
+				<box size="${green_plate_length} ${green_plate_width} ${green_plate_height}"/>
 			</geometry>
 			<origin xyz="0 0 0" rpy="0 0 0"/>
-			<material name="white">
+			<material name="green">
 				<color rgba="0 1 0 0.5"/>
 			</material>
@@ -63,5 +63,5 @@
 				<box size="${white_plate_width} ${white_plate_length} ${white_plate_height}"/>
 			</geometry>
-			<origin xyz="${white_plate_x_offset} 0 0" rpy="0 0 0"/>
+			<origin xyz="${-white_plate_x_offset} 0 0" rpy="0 0 0"/>
 			<material name="white">
 				<color rgba="1 1 1 0.5"/>
@@ -74,5 +74,5 @@
 				<box size="${stand_length} ${stand_width} ${stand_height}"/>
 			</geometry>
-			<origin xyz="0 0 0" rpy="${pi / 2} 0 ${pi / 2}"/>
+			<origin xyz="0 0 ${stand_height/2}" rpy="0 0 0"/>
 			<material name="white">
 				<color rgba="1 1 1 0.5"/>
@@ -83,5 +83,5 @@
 		<parent link="white_plate"/>
 		<child link="left_stand"/>
-		<origin xyz="0 ${white_plate_width / 2} ${-stand_length / 2}" rpy="0 0 0"/>
+		<origin xyz="0 ${white_plate_width / 2} 0" rpy="0 0 0"/>
 	</joint>
 	<link name="right_stand">
@@ -90,5 +90,5 @@
 				<box size="${stand_length} ${stand_width} ${stand_height}"/>
 			</geometry>
-			<origin xyz="0 0 0" rpy="${pi / 2} 0 ${pi / 2}"/>
+			<origin xyz="0 0 ${stand_height/2}" rpy="0 0 0"/>
 			<material name="white">
 				<color rgba="1 1 1 0.5"/>
@@ -96,8 +96,8 @@
 		</visual>
 	</link>
-	<joint name="white_plate_to_left_stand" type="fixed">
+	<joint name="white_plate_to_right_stand" type="fixed">
 		<parent link="white_plate"/>
 		<child link="right_stand"/>
-		<origin xyz="0 ${-white_plate_width / 2} ${-stand_length / 2}" rpy="0 0 0"/>
+		<origin xyz="0 ${-white_plate_width / 2} 0" rpy="0 0 0"/>
 	</joint>
 	<link name="header">
@@ -115,5 +115,5 @@
 		<parent link="white_plate"/>
 		<child link="header"/>
-		<origin xyz="${header_x_offset} 0 ${white_plate_height}" rpy="0 0 0"/>
+		<origin xyz="${header_x_offset} 0 ${header_z_offset}" rpy="0 0 0"/>
 	</joint>
 	<xacro:macro name="track" params="prefix reflect">

Commit message: collision added to be seen in gasebo

File: ROS/custom_src/orange_on_track/orange_on_track.xacro (robot description, xacro)
@@ -26,4 +26,12 @@
 	<xacro:property name="header_x_offset" value="0.10" />
 	<xacro:property name="header_z_offset" value="0.06" />
+	<xacro:macro name="default_inertial" params="mass">
+		<inertial>
+			<mass value="${mass}" />
+			<inertia ixx="1.0" ixy="0.0" ixz="0.0"
+				 iyy="1.0" iyz="0.0"
+				 izz="1.0" />
+		</inertial>
+	</xacro:macro>
 	<link name="base_link">
 		<visual>
@@ -36,4 +44,11 @@
 			</material>
 		</visual>
+		<collision>
+			<geometry>
+				<box size="${base_length} ${base_width} ${base_height}"/>
+			</geometry>
+			<origin xyz="0 0 0" rpy="0 0 0"/>
+		</collision>
+		<xacro:default_inertial mass="0.1"/>
 	</link>
 	<joint name="base_to_green_plate" type="fixed">
@@ -52,4 +67,5 @@
 			</material>
 		</visual>
+		<xacro:default_inertial mass="0.02"/>
 	</link>
 	<joint name="green_plate_to_white_plate" type="fixed">
@@ -68,4 +84,5 @@
 			</material>
 		</visual>
+		<xacro:default_inertial mass="0.05"/>
 	</link>
 	<link name="left_stand">
@@ -79,4 +96,5 @@
 			</material>
 		</visual>
+		<xacro:default_inertial mass="0.03"/>
 	</link>
 	<joint name="white_plate_to_left_stand" type="fixed">
@@ -95,4 +113,5 @@
 			</material>
 		</visual>
+		<xacro:default_inertial mass="0.03"/>
 	</link>
 	<joint name="white_plate_to_right_stand" type="fixed">
@@ -111,4 +130,5 @@
 			</material>
 		</visual>
+		<xacro:default_inertial mass="0.2"/>
 	</link>
 	<joint name="white_plate_to_header" type="fixed">
@@ -128,4 +148,5 @@
 				</material>
 			</visual>
+			<xacro:default_inertial mass="0.03"/>
 		</link>
 		<link name="${prefix}_fwd_wheel">
@@ -139,4 +160,5 @@
 				</material>
 			</visual>
+			<xacro:default_inertial mass="0.03"/>
 		</link>
 		<joint name="base_to_${prefix}_rear_wheel" type="continuous">
@@ -149,4 +171,8 @@
 			<child link="${prefix}_fwd_wheel"/>
 			<origin xyz="${wheel_x_offset} ${reflect*wheel_y_offset} 0" rpy="${pi / 2} 0 0"/>
+			<inertia
+				ixx="1.0" ixy="0.0" ixz="0.0"
+				iyy="1.0" iyz="0.0"
+				izz="1.0"/>
 		</joint>
 		<transmission name="base_to_${prefix}_rear_trans">
